Commit message: when parked very far, it dsent align

File: noetic_ws/src/gearfork_bot/urdf/gearfork_bot.urdf (robot description, URDF)
Before this commit: robot gearfork_bot, 8 links, 7 joints
Joints:
- joint motor_joint: limit lower=-0.88 upper=0.88 effort=5 velocity=1.0 -> lower=-0.88 upper=0.88 effort=5 velocity=10.0

Commit message: tricyle controller

File: noetic_ws/src/gearfork_bot/urdf/gearfork_bot.urdf (robot description, URDF)
Before this commit: robot gearfork_bot, 8 links, 7 joints
Links:
- link base_footprint: geometry collision mesh filename=package://gearfork_bot/meshes/base_footprint.STL; visual mesh filename=package://gearfork_bot/meshes/base_footprint.STL
- link base_link: geometry collision mesh filename=package://gearfork_bot/meshes/base_link.STL; visual mesh filename=package://gearfork_bot/meshes/base_link.STL
- link laser_link: geometry collision mesh filename=package://gearfork_bot/meshes/laser_link.STL; visual mesh filename=package://gearfork_bot/meshes/laser_link.STL
- link lroller_link: geometry collision mesh filename=package://gearfork_bot/meshes/lroller_link.STL; visual mesh filename=package://gearfork_bot/meshes/lroller_link.STL
- link motor_link: geometry collision mesh filename=package://gearfork_bot/meshes/motor_link.STL; visual mesh filename=package://gearfork_bot/meshes/motor_link.STL
- link rroller_link: geometry collision mesh filename=package://gearfork_bot/meshes/rroller_link.STL; visual mesh filename=package://gearfork_bot/meshes/rroller_link.STL
- link steering_link: geometry collision mesh filename=package://gearfork_bot/meshes/steering_link.STL; visual mesh filename=package://gearfork_bot/meshes/steering_link.STL
- link wheel_link: geometry collision mesh filename=package://gearfork_bot/meshes/wheel_link.STL; visual mesh filename=package://gearfork_bot/meshes/wheel_link.STL
Joints:
- joint motor_joint: limit (none) -> lower=-0.88 upper=0.88 effort=5 velocity=10.0; type continuous -> revolute
- joint wheel_joint: axis 0.0062645 -0.99998 0 -> 0.0062645 0.99998 0
